Commit message: log contact results, tweak fingers to be bigger

File: assets/hydro_panda.urdf (robot description, URDF)
Before this commit: robot panda, 12 links, 11 joints
Links:
- link panda_leftfinger: geometry collision box size=0.012 0.012 0.018; collision box size=0.012 0.012 0.018
- link panda_rightfinger: geometry collision box size=0.012 0.012 0.018; collision box size=0.012 0.012 0.018
